Commit message: ros_joint_4

File: gluon/urdf/gluon.urdf (robot description, URDF)
Before this commit: robot gluon, 8 links, 7 joints
Links:
- removed link 5_Link
- removed link 6_Link
Joints:
- removed joint axis_joint_5
- removed joint axis_joint_6

File: gluon/urdf/gluon_moveit_sim_pos.urdf (robot description, URDF)
Before this commit: robot gluon, 8 links, 7 joints
Links:
- removed link 5_Link
- removed link 6_Link
Joints:
- removed joint axis_joint_5
- removed joint axis_joint_6
